Commit message: parameter update

File: urdf/rg6_gripper.xacro (robot description, xacro)
@@ -218,5 +218,5 @@
 <link name="hand_tcp" />
 <joint name="hand_tcp_joint" type="fixed">
-  <origin xyz="0.031849 0 0.235" rpy="0 0 0" />
+  <origin xyz="0.036 0 0.21" rpy="0 0 0" />
   <parent link="g_main_1" />
   <child link="hand_tcp" />

Commit message: rename link names

File: urdf/rg6_gripper.xacro (robot description, xacro)
@@ -24,5 +24,5 @@
   </collision>
 </link>
-<link name="g_main_1">
+<link name="g_main">
   <inertial>
     <origin xyz="0.031843851343412694 -6.562152034605188e-05 0.0402561266087614" rpy="0 0 0"/>
@@ -33,5 +33,5 @@
     <origin xyz="0.031849 -1e-06 -0.04953" rpy="0 0 0"/>
     <geometry>
-      <mesh filename="package://rg6_gripper_description/meshes/g_main_1.stl" scale="0.001 0.001 0.001"/>
+      <mesh filename="package://rg6_gripper_description/meshes/g_main.stl" scale="0.001 0.001 0.001"/>
     </geometry>
     <material name="silver"/>
@@ -40,9 +40,9 @@
     <origin xyz="0.031849 -1e-06 -0.04953" rpy="0 0 0"/>
     <geometry>
-      <mesh filename="package://rg6_gripper_description/meshes/g_main_1.stl" scale="0.001 0.001 0.001"/>
-    </geometry>
-  </collision>
-</link>
-<link name="l_out_1">
+      <mesh filename="package://rg6_gripper_description/meshes/g_main.stl" scale="0.001 0.001 0.001"/>
+    </geometry>
+  </collision>
+</link>
+<link name="l_out">
   <inertial>
     <origin xyz="0.010442859349590227 -0.012799625869821 0.012792983853972317" rpy="0 0 0"/>
@@ -53,5 +53,5 @@
     <origin xyz="-0.023851 -0.012801 -0.13453" rpy="0 0 0"/>
     <geometry>
-      <mesh filename="package://rg6_gripper_description/meshes/l_out_1.stl" scale="0.001 0.001 0.001"/>
+      <mesh filename="package://rg6_gripper_description/meshes/l_out.stl" scale="0.001 0.001 0.001"/>
     </geometry>
     <material name="silver"/>
@@ -60,9 +60,9 @@
     <origin xyz="-0.023851 -0.012801 -0.13453" rpy="0 0 0"/>
     <geometry>
-      <mesh filename="package://rg6_gripper_description/meshes/l_out_1.stl" scale="0.001 0.001 0.001"/>
-    </geometry>
-  </collision>
-</link>
-<link name="r_out_1">
+      <mesh filename="package://rg6_gripper_description/meshes/l_out.stl" scale="0.001 0.001 0.001"/>
+    </geometry>
+  </collision>
+</link>
+<link name="r_out">
   <inertial>
     <origin xyz="-0.010522665986501832 -0.012799489922871823 0.012809246687502496" rpy="0 0 0"/>
@@ -73,5 +73,5 @@
     <origin xyz="0.023749 -0.012801 -0.13453" rpy="0 0 0"/>
     <geometry>
-      <mesh filename="package://rg6_gripper_description/meshes/r_out_1.stl" scale="0.001 0.001 0.001"/>
+      <mesh filename="package://rg6_gripper_description/meshes/r_out.stl" scale="0.001 0.001 0.001"/>
     </geometry>
     <material name="silver"/>
@@ -80,9 +80,9 @@
     <origin xyz="0.023749 -0.012801 -0.13453" rpy="0 0 0"/>
     <geometry>
-      <mesh filename="package://rg6_gripper_description/meshes/r_out_1.stl" scale="0.001 0.001 0.001"/>
-    </geometry>
-  </collision>
-</link>
-<link name="l_tip_1">
+      <mesh filename="package://rg6_gripper_description/meshes/r_out.stl" scale="0.001 0.001 0.001"/>
+    </geometry>
+  </collision>
+</link>
+<link name="l_tip">
   <inertial>
     <origin xyz="-0.01379426979129901 0.012430443916766657 0.03303967984911002" rpy="0 0 0"/>
@@ -93,5 +93,5 @@
     <origin xyz="-0.071235 0.012499 -0.19895" rpy="0 0 0"/>
     <geometry>
-      <mesh filename="package://rg6_gripper_description/meshes/l_tip_1.stl" scale="0.001 0.001 0.001"/>
+      <mesh filename="package://rg6_gripper_description/meshes/l_tip.stl" scale="0.001 0.001 0.001"/>
     </geometry>
     <material name="silver"/>
@@ -100,9 +100,9 @@
     <origin xyz="-0.071235 0.012499 -0.19895" rpy="0 0 0"/>
     <geometry>
-      <mesh filename="package://rg6_gripper_description/meshes/l_tip_1.stl" scale="0.001 0.001 0.001"/>
-    </geometry>
-  </collision>
-</link>
-<link name="r_tip_1">
+      <mesh filename="package://rg6_gripper_description/meshes/l_tip.stl" scale="0.001 0.001 0.001"/>
+    </geometry>
+  </collision>
+</link>
+<link name="r_tip">
   <inertial>
     <origin xyz="0.01379460286375201 0.012599371946431372 0.03303919214417522" rpy="0 0 0"/>
@@ -113,5 +113,5 @@
     <origin xyz="0.071133 0.012499 -0.199024" rpy="0 0 0"/>
     <geometry>
-      <mesh filename="package://rg6_gripper_description/meshes/r_tip_1.stl" scale="0.001 0.001 0.001"/>
+      <mesh filename="package://rg6_gripper_description/meshes/r_tip.stl" scale="0.001 0.001 0.001"/>
     </geometry>
     <material name="silver"/>
@@ -120,9 +120,9 @@
     <origin xyz="0.071133 0.012499 -0.199024" rpy="0 0 0"/>
     <geometry>
-      <mesh filename="package://rg6_gripper_description/meshes/r_tip_1.stl" scale="0.001 0.001 0.001"/>
-    </geometry>
-  </collision>
-</link>
-<link name="l_inner_1">
+      <mesh filename="package://rg6_gripper_description/meshes/r_tip.stl" scale="0.001 0.001 0.001"/>
+    </geometry>
+  </collision>
+</link>
+<link name="l_inner">
   <inertial>
     <origin xyz="0.021220873634115123 -0.00019955790008889003 0.02884270588361451" rpy="0 0 0"/>
@@ -133,5 +133,5 @@
     <origin xyz="-0.010551 -0.000101 -0.15763" rpy="0 0 0"/>
     <geometry>
-      <mesh filename="package://rg6_gripper_description/meshes/l_inner_1.stl" scale="0.001 0.001 0.001"/>
+      <mesh filename="package://rg6_gripper_description/meshes/l_inner.stl" scale="0.001 0.001 0.001"/>
     </geometry>
     <material name="silver"/>
@@ -140,9 +140,9 @@
     <origin xyz="-0.010551 -0.000101 -0.15763" rpy="0 0 0"/>
     <geometry>
-      <mesh filename="package://rg6_gripper_description/meshes/l_inner_1.stl" scale="0.001 0.001 0.001"/>
-    </geometry>
-  </collision>
-</link>
-<link name="r_inner_1">
+      <mesh filename="package://rg6_gripper_description/meshes/l_inner.stl" scale="0.001 0.001 0.001"/>
+    </geometry>
+  </collision>
+</link>
+<link name="r_inner">
   <inertial>
     <origin xyz="-0.021275767636285234 -0.00019955790008339296 0.02887567083082221" rpy="0 0 0"/>
@@ -153,5 +153,5 @@
     <origin xyz="0.010449 -0.000101 -0.15763" rpy="0 0 0"/>
     <geometry>
-      <mesh filename="package://rg6_gripper_description/meshes/r_inner_1.stl" scale="0.001 0.001 0.001"/>
+      <mesh filename="package://rg6_gripper_description/meshes/r_inner.stl" scale="0.001 0.001 0.001"/>
     </geometry>
     <material name="silver"/>
@@ -160,5 +160,5 @@
     <origin xyz="0.010449 -0.000101 -0.15763" rpy="0 0 0"/>
     <geometry>
-      <mesh filename="package://rg6_gripper_description/meshes/r_inner_1.stl" scale="0.001 0.001 0.001"/>
+      <mesh filename="package://rg6_gripper_description/meshes/r_inner.stl" scale="0.001 0.001 0.001"/>
     </geometry>
   </collision>
@@ -167,10 +167,10 @@
   <origin xyz="-0.031849 1e-06 0.04953" rpy="0 0 0"/>
   <parent link="base_link"/>
-  <child link="g_main_1"/>
+  <child link="g_main"/>
 </joint>
 <joint name="l_out" type="revolute">
   <origin xyz="0.0557 0.0128 0.085" rpy="0 0 0"/>
-  <parent link="g_main_1"/>
-  <child link="l_out_1"/>
+  <parent link="g_main"/>
+  <child link="l_out"/>
   <axis xyz="-0.0 1.0 0.0"/>
   <limit upper="0.610865" lower="-0.75" effort="100" velocity="100"/>
@@ -178,6 +178,6 @@
 <joint name="r_out" type="revolute">
   <origin xyz="0.0081 0.0128 0.085" rpy="0 0 0"/>
-  <parent link="g_main_1"/>
-  <child link="r_out_1"/>
+  <parent link="g_main"/>
+  <child link="r_out"/>
   <axis xyz="-0.0 1.0 0.0"/>
   <limit upper="0.523599" lower="-0.610865" effort="100" velocity="100"/>
@@ -186,6 +186,6 @@
 <joint name="l_tip" type="revolute">
   <origin xyz="0.047384 -0.0253 0.06442" rpy="0 0 0"/>
-  <parent link="l_out_1"/>
-  <child link="l_tip_1"/>
+  <parent link="l_out"/>
+  <child link="l_tip"/>
   <axis xyz="0.0 -1.0 0.0"/>
   <limit upper="0.610865" lower="-0.523599" effort="100" velocity="100"/>
@@ -194,6 +194,6 @@
 <joint name="r_tip" type="revolute">
   <origin xyz="-0.047384 -0.0253 0.064494" rpy="0 0 0"/>
-  <parent link="r_out_1"/>
-  <child link="r_tip_1"/>
+  <parent link="r_out"/>
+  <child link="r_tip"/>
   <axis xyz="0.0 -1.0 0.0"/>
   <limit upper="0.523599" lower="-0.610865" effort="100" velocity="100"/>
@@ -202,6 +202,6 @@
 <joint name="l_passive" type="revolute">
   <origin xyz="0.0424 0.0001 0.1081" rpy="0 0 0"/>
-  <parent link="g_main_1"/>
-  <child link="l_inner_1"/>
+  <parent link="g_main"/>
+  <child link="l_inner"/>
   <axis xyz="0.0 -1.0 0.0"/>
   <limit upper="0.523599" lower="-0.610865" effort="100" velocity="100"/>
@@ -210,6 +210,6 @@
 <joint name="r_passive" type="revolute">
   <origin xyz="0.0214 0.0001 0.1081" rpy="0 0 0"/>
-  <parent link="g_main_1"/>
-  <child link="r_inner_1"/>
+  <parent link="g_main"/>
+  <child link="r_inner"/>
   <axis xyz="-0.0 1.0 -0.0"/>
   <limit upper="0.523599" lower="-0.610865" effort="100" velocity="100"/>
@@ -219,5 +219,5 @@
 <joint name="hand_tcp_joint" type="fixed">
   <origin xyz="0.036 0 0.21" rpy="0 0 0" />
-  <parent link="g_main_1" />
+  <parent link="g_main" />
   <child link="hand_tcp" />
   <axis xyz="-0.0 1.0 -0.0"/>
